File: DRV-24to12-BrushedMotorDriver.kicad_sch (KiCad schematic)
At the start: 29 parts, among them J1 Conn_01x02, J2 Conn_01x02, J3 Conn_01x05_Pin, U1 DRV8801PWP, U2 TPS5430DDA, U4 AMS1117-3.3

Commit message: Layout done
Parts:
- removed C5: 100uF 25V, Capacitor_SMD:CP_Elec_6.3x7.7, symbol Device:C_Polarized
- removed C8: C_Polarized, Capacitor_SMD:CP_Elec_5x5.4, symbol Device:C_Polarized
- removed J2: Conn_01x02, Connector_AMASS:AMASS_XT30U-M_1x02_P5.0mm_Vertical, symbol Connector_Generic:Conn_01x02
- removed J3: Conn_01x05_Pin, symbol Connector:Conn_01x05_Pin
- removed U4: AMS1117-3.3, Package_TO_SOT_SMD:SOT-223-3_TabPin2, symbol Regulator_Linear:AMS1117-3.3
- added C5: 2.2uF, Capacitor_SMD:C_1206_3216Metric_Pad1.33x1.80mm_HandSolder, symbol Device:C
- added D2, D3: SS34, Diode_SMD:D_SMA, symbol Device:D_Schottky
- added J3: Conn_02x04_Odd_Even, Connector_PinHeader_2.54mm:PinHeader_2x04_P2.54mm_Vertical_SMD, symbol Connector_Generic:Conn_02x04_Odd_Even
- added R5: 0R 1A, Capacitor_SMD:C_0603_1608Metric, symbol Device:R
- added R6, R7: 0R 1A, Capacitor_SMD:C_1206_3216Metric, symbol Device:R
- added TP1: PWR_IN+, TestPoint:TestPoint_Pad_4.0x4.0mm, symbol Connector:TestPoint
- added TP2: PWR_IN-, TestPoint:TestPoint_Pad_4.0x4.0mm, symbol Connector:TestPoint
- added U3: ME6211C33M5, Package_TO_SOT_SMD:SOT-23-5, symbol Regulator_Linear:AP131-33
- C1, C2, C3, C4: footprint (none) -> Capacitor_SMD:C_0603_1608Metric
- J1: footprint (none) -> Connector_JST:JST_PH_B2B-PH-SM4-TB_1x02-1MP_P2.00mm_Vertical; symbol Connector_Generic:Conn_01x02 -> Connector_Generic_MountingPin:Conn_01x02_MountingPin
- U1: footprint Package_SO:HTSSOP-16-1EP_4.4x5mm_P0.65mm_EP3.4x5mm_Mask3x3mm_ThermalVias -> Package_SO:HTSSOP-16-1EP_4.4x5mm_P0.65mm_EP3.4x5mm_Mask2.46x2.31mm
- U2: footprint Package_SO:TI_SO-PowerPAD-8_ThermalVias -> Package_SO:TI_SO-PowerPAD-8
Connections:
- net +12V: now also U3.1 (IN), U3.3 (EN)
- net +24V: now also TP1.1
- net +3V3: now also C5.2, U3.5 (OUT)
- net GND: now also J1.MP (MountPin), C5.1, D2.2 (A), D3.2 (A), J3.2 (Pin_2), J3.4 (Pin_4), J3.6 (Pin_6), J3.8 (Pin_8), TP2.1, U3.2 (GND)
- net MOTOR+: now also J1.2 (Pin_2), D2.1 (K), R7.2; no longer J1.1 (Pin_1), U1.7 (OUT+)
- net MOTOR-: now also J1.1 (Pin_1), D3.1 (K), R5.2; no longer J1.2 (Pin_2), U1.10 (OUT-)
- net MOTOR_RUN: now also J3.1 (Pin_1)
- net NFAULT: now also J3.7 (Pin_7)
- net PHASE_CTRL: now also J3.5 (Pin_5)
- net VPROPI: now also J3.3 (Pin_3)
- new net: R6.1, U1.7 (OUT+)
- new net: R6.2, R7.1
- new net: R5.1, U1.10 (OUT-)
- no-connect marks 5 -> 6
Other:
- moved on the sheet: C10

Commit message: layout2
Parts:
- H1, H2, H3, H4: footprint MountingHole:MountingHole_3.2mm_M3_Pad_Via -> MountingHole:MountingHole_3.2mm_M3_Pad_TopOnly
- R2: value 0 -> 4.7K
- R5: footprint Capacitor_SMD:C_0603_1608Metric -> Resistor_SMD:R_1206_3216Metric
- R6, R7: footprint Capacitor_SMD:C_1206_3216Metric -> Resistor_SMD:R_1206_3216Metric
Connections:
- net NFAULT: now also J3.5 (Pin_5); no longer J3.7 (Pin_7)
- net PHASE_CTRL: now also J3.3 (Pin_3); no longer J3.5 (Pin_5)
- net VPROPI: now also J3.7 (Pin_7); no longer J3.3 (Pin_3)
Changed lines of the file:
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@@
+    (stroke (width 0) (type default))
+  )
+  (wire (pts (xy 214.63 137.16) (xy 217.17 137.16))
     (stroke (width 0) (type default))
   )
@@
     (stroke (width 0) (type default))
   )
+  (wire (pts (xy 214.63 142.24) (xy 217.17 142.24))
+    (stroke (width 0) (type default))
+  )
   (wire (pts (xy 76.2 93.98) (xy 80.01 93.98))
     (stroke (width 0) (type default))
@@
     (stroke (width 0) (type default))
   )
-  (wire (pts (xy 214.63 142.24) (xy 217.17 142.24))
+  (wire (pts (xy 214.63 139.7) (xy 217.17 139.7))
     (stroke (width 0) (type default))
   )
@@
     (stroke (width 0) (type default))
   )
-  (wire (pts (xy 214.63 137.16) (xy 217.17 137.16))
-    (stroke (width 0) (type default))
-  )
   (wire (pts (xy 97.79 66.04) (xy 95.25 66.04))
     (stroke (width 0) (type default))
@@
   )
   (wire (pts (xy 229.87 142.24) (xy 232.41 142.24))
-    (stroke (width 0) (type default))
-  )
-  (wire (pts (xy 214.63 139.7) (xy 217.17 139.7))
     (stroke (width 0) (type default))
   )
@@
     (effects (font (size 1.27 1.27)) (justify left))
   )
-  (hierarchical_label "NFAULT" (shape output) (at 214.63 142.24 180) (fields_autoplaced)
+  (hierarchical_label "NFAULT" (shape output) (at 214.63 139.7 180) (fields_autoplaced)
     (effects (font (size 1.27 1.27)) (justify right))
   )
-  (hierarchical_label "PHASE_CTRL" (shape input) (at 214.63 139.7 180) (fields_autoplaced)
+  (hierarchical_label "PHASE_CTRL" (shape input) (at 214.63 137.16 180) (fields_autoplaced)
     (effects (font (size 1.27 1.27)) (justify right))
   )
@@
     (effects (font (size 1.27 1.27)) (justify right))
   )
-  (hierarchical_label "VPROPI" (shape output) (at 214.63 137.16 180) (fields_autoplaced)
+  (hierarchical_label "VPROPI" (shape output) (at 214.63 142.24 180) (fields_autoplaced)
     (effects (font (size 1.27 1.27)) (justify right))
   )
@@
       (effects (font (size 1.27 1.27)) (justify left))
     )
-    (property "Footprint" "MountingHole:MountingHole_3.2mm_M3_Pad_Via" (at 151.13 176.53 0)
+    (property "Footprint" "MountingHole:MountingHole_3.2mm_M3_Pad_TopOnly" (at 151.13 176.53 0)
       (effects (font (size 1.27 1.27)) hide)
     )
@@
       (effects (font (size 1.27 1.27)))
     )
-    (property "Footprint" "Capacitor_SMD:C_1206_3216Metric" (at 118.11 38.608 90)
+    (property "Footprint" "Resistor_SMD:R_1206_3216Metric" (at 118.11 38.608 90)
       (effects (font (size 1.27 1.27)) hide)
     )
@@
       (effects (font (size 1.27 1.27)))
     )
-    (property "Footprint" "Capacitor_SMD:C_1206_3216Metric" (at 127 38.608 90)
+    (property "Footprint" "Resistor_SMD:R_1206_3216Metric" (at 127 38.608 90)
       (effects (font (size 1.27 1.27)) hide)
     )
@@
       (effects (font (size 1.27 1.27)))
     )
-    (property "Footprint" "Capacitor_SMD:C_0603_1608Metric" (at 118.11 41.148 90)
+    (property "Footprint" "Resistor_SMD:R_1206_3216Metric" (at 118.11 41.148 90)
       (effects (font (size 1.27 1.27)) hide)
     )
@@
       (effects (font (size 1.27 1.27)))
     )
-    (property "Value" "0" (at 63.5 62.23 90)
+    (property "Value" "4.7K" (at 63.5 62.23 90)
       (effects (font (size 1.27 1.27)))
     )
@@
       (effects (font (size 1.27 1.27)) (justify left))
     )
-    (property "Footprint" "MountingHole:MountingHole_3.2mm_M3_Pad_Via" (at 151.13 170.18 0)
+    (property "Footprint" "MountingHole:MountingHole_3.2mm_M3_Pad_TopOnly" (at 151.13 170.18 0)
       (effects (font (size 1.27 1.27)) hide)
     )
@@
       (effects (font (size 1.27 1.27)) (justify left))
     )
-    (property "Footprint" "MountingHole:MountingHole_3.2mm_M3_Pad_Via" (at 151.13 182.88 0)
+    (property "Footprint" "MountingHole:MountingHole_3.2mm_M3_Pad_TopOnly" (at 151.13 182.88 0)
       (effects (font (size 1.27 1.27)) hide)
     )
@@
       (effects (font (size 1.27 1.27)) (justify left))
     )
-    (property "Footprint" "MountingHole:MountingHole_3.2mm_M3_Pad_Via" (at 151.13 189.23 0)
-      (effects (font (size 1.27 1.27)) hide)
-    )
+    (property "Footprint" "MountingHole:MountingHole_3.2mm_M3_Pad_TopOnly" (at 151.13 189.23 0)
+      (effects (font (size 1.27 1.27)) hide)
+    )

Commit message: ver1.0 done
Parts:
- added C8: 10nF, Capacitor_SMD:C_0603_1608Metric, symbol Device:C
- added R10: 0R 1A, Resistor_SMD:R_1206_3216Metric, symbol Device:R
- added R8: 22R, Resistor_SMD:R_0603_1608Metric, symbol Device:R
- added R9: 0R, Resistor_SMD:R_1206_3216Metric, symbol Device:R
- added U4: LM358, Package_SO:SOIC-8_3.9x4.9mm_P1.27mm, symbol Amplifier_Operational:LM358
- U3: value ME6211C33M5 -> ME6214C33M5G
Connections:
- net +12V: now also R10.1; no longer C10.2, U3.1 (IN), U3.3 (EN)
- net +3V3: now also C8.2, U4.8 (V+)
- net GND: now also C8.1, U4.4 (V-)
- net VPROPI: now also U4.3 (+); no longer J3.7 (Pin_7)
- new net: R9.1, U4.1, U4.2 (-)
- new net: R8.1, R9.2
- new net: C10.2, R10.2, U3.1 (IN), U3.3 (EN)
- new net VPROPI_AMP: J3.7 (Pin_7), R8.2
- no-connect marks 6 -> 9
